Commit message: Update urdf

File: description/wheels/kelo_drive_mid.xacro (robot description, xacro)
@@ -32,5 +32,5 @@
 -->
 <robot xmlns:xacro="http://www.ros.org/wiki/xacro">
-    <xacro:macro name="kelo_drive" params="name parent *origin movable_joints:=true">
+    <xacro:macro name="kelo_drive_mid" params="name parent *origin movable_joints:=true">
         <xacro:include filename="$(find skratch_description)/description/wheels/kelo_drive_wheel.xacro"/>
         <link name="${name}_pivot_link">
@@ -62,5 +62,5 @@
                 <parent link="${parent}"/>
                 <child link="${name}_pivot_link" />
-                <dynamics damping="0.1" friction="0.05"/>
+                <dynamics damping="1.0" friction="0.1"/>
                 <limit effort="2.0" velocity="1.0"/>
             </joint>
