Commit message: Adding URDF for classic

File: sensor_mounts/lidar_mount.xacro (robot description, xacro)
@@ -8,6 +8,6 @@
 -->
 <robot name="lidar_mount" xmlns:xacro="http://www.ros.org/wiki/xacro">
-    <xacro:macro name="lidar_mount" params="name parent *origin">
-        <xacro:include filename="$(find skratch_description)/description/sensors/hokuyo_urg_04lx_ug01.xacro"/>
+    <xacro:macro name="lidar_mount" params="name parent *origin ros_topic update_rate min_angle max_angle">
+        <xacro:include filename="$(find skratch_description)/sensors/hokuyo_urg_04lx_ug01.xacro"/>
         <link name="${name}_lidar_mount">
             <inertial>
@@ -40,5 +40,5 @@
             <child link="${name}_lidar_mount"/>
         </joint>
-        <xacro:hokuyo_urg_lidar name="${name}_hokuyo_urg_lidar" parent="${name}_lidar_mount">
+        <xacro:hokuyo_urg_lidar name="${name}_hokuyo_urg_lidar" parent="${name}_lidar_mount" ros_topic="${ros_topic}" update_rate="${update_rate}" min_angle="${min_angle}" max_angle="${max_angle}">
             <origin xyz="0.045 -0.045 -0.1" rpy="3.14 0.0 -0.77"/>
         </xacro:hokuyo_urg_lidar>

File: sensors/hokuyo_urg_04lx_ug01.xacro (robot description, xacro)
@@ -8,5 +8,5 @@
 -->
 <robot name="hokuyo_urg_lidar" xmlns:xacro="http://www.ros.org/wiki/xacro">
-    <xacro:macro name="hokuyo_urg_lidar" params="name parent *origin">
+    <xacro:macro name="hokuyo_urg_lidar" params="name ros_topic update_rate min_angle max_angle parent *origin">
         <link name="${name}_hokuyo_urg_lidar_link">
             <inertial>
@@ -31,36 +31,39 @@
             </collision>
         </link>
-        <gazebo reference="${name}_hokuyo_urg_lidar_link">
-            <material>Gazebo/Black</material>
-            <sensor type="gpu_lidar" name="${name}_hokuyo_urg_lidar">
-                <pose>0 0 0.06 0 0 0</pose>
-                <visualize>true</visualize>
-                <update_rate>10</update_rate>
-                <lidar>
-                    <scan>
-                        <horizontal>
-                            <samples>682</samples>
-                            <resolution>1</resolution>
-                            <min_angle>-2.35619449</min_angle>
-                            <!-- -135° in rad -->
-                            <max_angle>2.35619449</max_angle>
-                            <!-- 135° in rad -->
-                        </horizontal>
-                    </scan>
-                    <range>
-                        <min>0.06</min>
-                        <max>5.6</max>
-                        <resolution>0.001</resolution>
-                    </range>
-                    <noise>
-                        <type>gaussian</type>
-                        <mean>0.0</mean>
-                        <stddev>0.005</stddev>
-                    </noise>
-                </lidar>
-                <topic>/${name}_scan</topic>
-                <gz_frame_id>${name}_hokuyo_urg_lidar_link</gz_frame_id>
-            </sensor>
-        </gazebo>
+    <!-- Gazebo Classic sensor plugin -->
+    <gazebo reference="${name}_link">
+      <sensor name="${name}" type="ray">
+        <update_rate>${update_rate}</update_rate>
+        <pose>0 0 0 0 0 0</pose>
+        <visualize>true</visualize>
+        <ray>
+          <scan>
+            <horizontal>
+              <samples>150</samples>
+              <resolution>1.0</resolution>
+              <min_angle>${min_angle}</min_angle>
+              <max_angle>${max_angle}</max_angle>
+            </horizontal>
+          </scan>
+          <range>
+            <min>0.05</min>
+            <max>5.6</max>
+            <resolution>0.36</resolution>
+          </range>
+          <noise>
+            <type>gaussian</type>
+            <mean>0.0</mean>
+            <stddev>0.01</stddev>
+          </noise>
+        </ray>
+        <plugin name="gazebo_ros_${name}_controller" filename="libgazebo_ros_ray_sensor.so">
+          <ros>
+            <remapping>~/out:=${ros_topic}</remapping>
+          </ros>
+          <output_type>sensor_msgs/LaserScan</output_type>
+          <frame_name>${name}_link</frame_name>
+        </plugin>
+      </sensor>
+    </gazebo>
         <joint name="${name}_hokuyo_urg_lidar_mount_joint" type="fixed">
             <xacro:insert_block name="origin"/>

File: wheels/kelo_drive_mid.urdf.xacro (robot description, xacro)
@@ -32,43 +32,42 @@
 -->
 <robot xmlns:xacro="http://www.ros.org/wiki/xacro">
-    <xacro:macro name="kelo_drive_wheel" params="name parent *origin movable_joints:=true">
-        <link name="${name}_link">
+    <xacro:macro name="kelo_drive_mid" params="name parent *origin movable_joints:=true">
+        <xacro:include filename="$(find skratch_description)/wheels/common.xacro" />
+        <xacro:include filename="$(find skratch_description)/wheels/kelo_drive_wheel.urdf.xacro" />
+        <!-- PIVOT Link-->
+        <link name="${name}_pivot_link">
             <visual>
                 <origin xyz="0 0 0" rpy="0 0 0"/>
                 <geometry>
-                    <mesh filename="file://$(find skratch_description)/meshes/wheels/kelo_drive_hub_wheel.dae" scale="1 1 1"/>
+                    <mesh filename="file://$(find skratch_description)/meshes/kelo_drive/kelo_drive_mid_part.dae" scale="1 1 1"/>
                 </geometry>
-                <material name="black">
-                    <color rgba="0.0 0.0 0.0 1.0"/>
-                </material>
             </visual>
             <collision>
                 <origin xyz="0 0 0" rpy="0 0 0"/>
                 <geometry>
-                    <mesh filename="file://$(find skratch_description)/meshes/wheels/kelo_drive_wheel.dae" scale="1 1 1"/>
+                    <mesh filename="file://$(find skratch_description)/meshes/kelo_drive/kelo_drive_mid_part.dae" scale="1 1 1"/>
                 </geometry>
             </collision>
             <inertial>
-                <origin xyz="0 0 0" rpy="0 0 0"/>
-                <mass value="1.56317"/>
-                <inertia ixx="0.00101253363" ixy="0.00000000000" ixz="0.00000001020" iyy="0.00157998524" iyz="-0.00000055474" izz="0.00101282739"/>
+                <origin xyz="0.00023 -0.00095 0.04843" rpy="0 0 0"/>
+                <mass value="1.46273"/>
+                <inertia ixx="0.00302046423" ixy="0.00000851844" ixz="0.00001188180" iyy="0.00326495472" iyz="0.00001855408" izz="0.00386072964"/>
             </inertial>
         </link>
-        <gazebo reference="${name}_link">
-            <material>Gazebo/Black</material>
-        </gazebo>
+        <!-- PIVOT continous or fixed-->
         <xacro:if value="${movable_joints}">
-            <joint name="${name}_joint" type="continuous">
+            <joint name="${name}_pivot_joint" type="continuous">
                 <xacro:insert_block name="origin" />
-                <axis xyz="0 1 0"/>
+                <axis xyz="0 0 1"/>
                 <parent link="${parent}"/>
-                <child link="${name}_link" />
+                <child link="${name}_pivot_link" />
+                <limit effort="2.0" velocity="1.0"/>
             </joint>
-            <transmission name="${name}_transmission">
+            <transmission name="${name}_pivot_transmission">
                 <type>transmission_interface/SimpleTransmission</type>
-                <joint name="${name}_joint">
+                <joint name="${name}_pivot_joint">
                     <hardwareInterface>hardware_interface/EffortJointInterface</hardwareInterface>
                 </joint>
-                <actuator name="${name}_motor">
+                <actuator name="${name}_pivot_motor">
                     <hardwareInterface>hardware_interface/EffortJointInterface</hardwareInterface>
                     <mechanicalReduction>1</mechanicalReduction>
@@ -77,10 +76,19 @@
         </xacro:if>
         <xacro:unless value="${movable_joints}">
-            <joint name="${name}_joint" type="fixed">
+            <joint name="${name}_pivot_joint" type="fixed">
                 <xacro:insert_block name="origin" />
+                <axis xyz="0 0 1"/>
                 <parent link="${parent}"/>
-                <child link="${name}_link" />
+                <child link="${name}_pivot_link" />
             </joint>
         </xacro:unless>
+        <!-- LEFT HUB WHEEL -->
+        <xacro:kelo_drive_wheel name="${name}_left_hub_wheel" parent="${name}_pivot_link" movable_joints="${movable_joints}">
+            <origin xyz="-0.01 0.039326 0.001514" rpy="0 0 0.0"/>
+        </xacro:kelo_drive_wheel>
+        <!-- RIGHT HUB WHEEL -->
+        <xacro:kelo_drive_wheel name="${name}_right_hub_wheel" parent="${name}_pivot_link" movable_joints="${movable_joints}">
+            <origin xyz="-0.01 -0.039326 0.001514" rpy="0 0 0.0"/>
+        </xacro:kelo_drive_wheel>
     </xacro:macro>
 </robot>

File: wheels/kelo_drive_wheel.urdf.xacro (robot description, xacro)
@@ -5,6 +5,4 @@
 Author:
 Sushant Chavan
-Maintainer:
-Chaitanya Gumudala
 This software is published under a dual-license: GNU Lesser General Public
 License LGPL 2.1 and BSD license. The dual-license implies that users of this
@@ -32,43 +30,19 @@
 -->
 <robot xmlns:xacro="http://www.ros.org/wiki/xacro">
-    <xacro:macro name="kelo_drive_mid" params="name parent *origin movable_joints:=true">
-        <xacro:include filename="$(find skratch_description)/description/wheels/kelo_drive_wheel.xacro"/>
-        <link name="${name}_pivot_link">
-            <visual>
-                <origin xyz="0 0 0.0" rpy="0 0 0"/>
-                <geometry>
-                    <mesh filename="file://$(find skratch_description)/meshes/wheels/kelo_drive_mid_part.dae" scale="1 1 1"/>
-                </geometry>
-                <material name="light_grey">
-                    <color rgba="0.2 0.2 0.2 1.0"/>
-                </material>
-            </visual>
-            <collision>
-                <origin xyz="0 0 0.0" rpy="0 0 0"/>
-                <geometry>
-                    <mesh filename="file://$(find skratch_description)/meshes/wheels/kelo_drive_mid_part.dae" scale="1 1 1"/>
-                </geometry>
-            </collision>
-            <inertial>
-                <origin xyz="0.00023 -0.00095 0.024" rpy="0 0 0"/>
-                <mass value="1.46273"/>
-                <inertia ixx="0.00302046423" ixy="0.00" ixz="0.0" iyy="0.00326495472" iyz="0.0" izz="0.00386072964"/>
-            </inertial>
-        </link>
+    <xacro:macro name="kelo_drive_wheel" params="name parent *origin movable_joints:=true">
+        <xacro:include filename="$(find skratch_description)/wheels/common.xacro" />
         <xacro:if value="${movable_joints}">
-            <joint name="${name}_pivot_joint" type="continuous">
+            <joint name="${name}_joint" type="continuous">
                 <xacro:insert_block name="origin" />
-                <axis xyz="0 0 1"/>
+                <axis xyz="0 1 0"/>
                 <parent link="${parent}"/>
-                <child link="${name}_pivot_link" />
-                <dynamics damping="1.0" friction="0.1"/>
-                <limit effort="2.0" velocity="1.0"/>
+                <child link="${name}_link" />
             </joint>
-            <transmission name="${name}_pivot_transmission">
+            <transmission name="${name}_transmission">
                 <type>transmission_interface/SimpleTransmission</type>
-                <joint name="${name}_pivot_joint">
+                <joint name="${name}_joint">
                     <hardwareInterface>hardware_interface/EffortJointInterface</hardwareInterface>
                 </joint>
-                <actuator name="${name}_pivot_motor">
+                <actuator name="${name}_motor">
                     <hardwareInterface>hardware_interface/EffortJointInterface</hardwareInterface>
                     <mechanicalReduction>1</mechanicalReduction>
@@ -76,19 +50,31 @@
             </transmission>
         </xacro:if>
-        <xacro:unless value ="${movable_joints}">
-            <joint name="${name}_pivot_joint" type="fixed">
+        <xacro:unless value="${movable_joints}">
+            <joint name="${name}_joint" type="fixed">
                 <xacro:insert_block name="origin" />
+                <axis xyz="0 1 0"/>
                 <parent link="${parent}"/>
-                <child link="${name}_pivot_link" />
+                <child link="${name}_link" />
             </joint>
         </xacro:unless>
-        <!-- LEFT HUB WHEEL -->
-        <xacro:kelo_drive_wheel name="${name}_left_hub_wheel" parent="${name}_pivot_link" movable_joints="${movable_joints}">
-            <origin xyz="-0.0 0.039326 0.001514" rpy="0 0 0.0"/>
-        </xacro:kelo_drive_wheel>
-        <!-- RIGHT HUB WHEEL -->
-        <xacro:kelo_drive_wheel name="${name}_right_hub_wheel" parent="${name}_pivot_link" movable_joints="${movable_joints}">
-            <origin xyz="-0.0 -0.039326 0.001514" rpy="0 0 0.0"/>
-        </xacro:kelo_drive_wheel>
+        <link name="${name}_link">
+            <visual>
+                <origin xyz="0 0 0" rpy="0 0 0"/>
+                <geometry>
+                    <mesh filename="file://$(find skratch_description)/meshes/kelo_drive/kelo_drive_wheel.stl" scale="1 1 1"/>
+                </geometry>
+            </visual>
+            <collision>
+                <origin xyz="0 0 0" rpy="0 0 0"/>
+                <geometry>
+                    <mesh filename="file://$(find skratch_description)/meshes/kelo_drive/kelo_drive_wheel.stl" scale="1 1 1"/>
+                </geometry>
+            </collision>
+             <inertial>
+                <origin xyz="0 0 0" rpy="0 0 0"/>
+                <mass value="1.56317"/>
+                <inertia ixx="0.00101253363" ixy="0.00000000000" ixz="0.00000001020" iyy="0.00157998524" iyz="-0.00000055474" izz="0.00101282739"/>
+            </inertial>
+        </link>
     </xacro:macro>
 </robot>

Commit message: Updating URDF propely with Lidar

File: sensor_mounts/lidar_mount.xacro (robot description, xacro)
@@ -8,5 +8,5 @@
 -->
 <robot name="lidar_mount" xmlns:xacro="http://www.ros.org/wiki/xacro">
-    <xacro:macro name="lidar_mount" params="name parent *origin ros_topic update_rate min_angle max_angle">
+    <xacro:macro name="lidar_mount" params="name parent *origin">
         <xacro:include filename="$(find skratch_description)/sensors/hokuyo_urg_04lx_ug01.xacro"/>
         <link name="${name}_lidar_mount">
@@ -40,7 +40,17 @@
             <child link="${name}_lidar_mount"/>
         </joint>
-        <xacro:hokuyo_urg_lidar name="${name}_hokuyo_urg_lidar" parent="${name}_lidar_mount" ros_topic="${ros_topic}" update_rate="${update_rate}" min_angle="${min_angle}" max_angle="${max_angle}">
-            <origin xyz="0.045 -0.045 -0.1" rpy="3.14 0.0 -0.77"/>
-        </xacro:hokuyo_urg_lidar>
+        <xacro:if value="$(arg use_sim)">
+            <xacro:hokuyo_urg_lidar
+                name="${name}_lidar"
+                ros_topic="/${name}_scan"
+                update_rate="10"
+                min_angle="-1.57"
+                max_angle="2.35" />
+            <joint name="${name}_lidar_joint" type="fixed">
+                <origin xyz="0.048 -0.048 -0.10" rpy="0.0 0.0 -0.785"/>
+                <parent link="${name}_lidar_mount"/>
+                <child link="${name}_lidar_stl_link"/>
+            </joint>
+        </xacro:if>
     </xacro:macro>
 </robot>

File: sensors/hokuyo_urg_04lx_ug01.xacro (robot description, xacro)
@@ -1,39 +1,51 @@
 <?xml version="1.0"?>
-<!--
-Copyright (c) 2025
-b-it-bots
-Hochschule Bonn-Rhein-Sieg
-Authors:
-Chaitanya Gumudala
--->
-<robot name="hokuyo_urg_lidar" xmlns:xacro="http://www.ros.org/wiki/xacro">
-    <xacro:macro name="hokuyo_urg_lidar" params="name ros_topic update_rate min_angle max_angle parent *origin">
-        <link name="${name}_hokuyo_urg_lidar_link">
-            <inertial>
-                <mass value="0.16"/>
-                <origin xyz="0 0 0.035" rpy="0 0 0"/>
-                <inertia ixx="0.0001563" iyy="0.0001563" izz="0.0001333" ixy="0.0" ixz="0.0" iyz="0.0"/>
-            </inertial>
-            <visual>
-                <origin xyz="0.0 0.0 0.0" rpy="0.0 0.0 0.0" />
-                <geometry>
-                    <mesh filename="file://$(find skratch_description)/meshes/sensors/Hokuyo_URG_04LX_UG01.stl" scale="1 1 1"/>
-                </geometry>
-                <material name="Black">
-                    <color rgba="0.0 0.0 0.0 1.0"/>
-                </material>
-            </visual>
-            <collision>
-                <origin xyz="0.0 0.0 0.0" rpy="0.0 0.0 0.0" />
-                <geometry>
-                    <mesh filename="file://$(find skratch_description)/meshes/sensors/Hokuyo_URG_04LX_UG01.stl" scale="1 1 1"/>
-                </geometry>
-            </collision>
-        </link>
-    <!-- Gazebo Classic sensor plugin -->
-    <gazebo reference="${name}_link">
-      <sensor name="${name}" type="ray">
+<robot name="lidar_robot" xmlns:xacro="http://www.ros.org/wiki/xacro">
+  <xacro:macro name="hokuyo_urg_lidar" params="name ros_topic update_rate min_angle max_angle">
+    <!-- Link with STL geometry -->
+    <link name="${name}_stl_link">
+      <inertial>
+        <mass value="0.16" />
+        <origin xyz="0.0 0.0 0.035" rpy="0.0 0.0 0.0" />
+        <inertia ixx="0.0001563" iyy="0.0001563" izz="0.0001333" ixy="0.0" ixz="0.0" iyz="0.0"/>
+      </inertial>
+      <visual>
+        <origin xyz="0.0 0.0 0.0" rpy="0.0 3.14 3.14" />
+        <geometry>
+          <mesh filename="file://$(find skratch_description)/meshes/sensors/Hokuyo_URG_04LX_UG01.stl" scale="1 1 1"/>
+        </geometry>
+        <material name="Black">
+          <color rgba="0 0 0 1"/>
+        </material>
+      </visual>
+      <collision>
+        <origin xyz="0.0 0.0 0.0" rpy="0.0 3.14 3.14" />
+        <geometry>
+          <mesh filename="file://$(find skratch_description)/meshes/sensors/Hokuyo_URG_04LX_UG01.stl" scale="1 1 1"/>
+        </geometry>
+      </collision>
+    </link>
+    <!-- Gazebo material -->
+    <gazebo reference="${name}_stl_link">
+      <material>Gazebo/Black</material>
+    </gazebo>
+     <!-- Child link only for the laser rays -->
+    <link name="${name}_ray_link">
+      <inertial>
+        <mass value="0.001"/>
+        <origin xyz="0 0 0" rpy="0 0 0"/>
+        <inertia ixx="0.000001" iyy="0.000001" izz="0.000001" ixy="0.0" ixz="0.0" iyz="0.0"/>
+      </inertial>
+    </link>
+    <!-- ↓↓↓ Move ray start point 5 cm below STL origin ↓↓↓ -->
+    <joint name="${name}_ray_joint" type="fixed">
+      <origin xyz="0 0 -0.05" rpy="0 0 0"/>
+      <parent link="${name}_stl_link"/>
+      <child link="${name}_ray_link"/>
+    </joint>
+    <!-- Gazebo sensor plugin -->
+    <gazebo reference="${name}_ray_link">
+      <sensor name="${name}_sensor" type="ray">
         <update_rate>${update_rate}</update_rate>
-        <pose>0 0 0 0 0 0</pose>
+        <pose>0 0 0.0 0 0 0</pose>
         <visualize>true</visualize>
         <ray>
@@ -62,13 +74,8 @@
           </ros>
           <output_type>sensor_msgs/LaserScan</output_type>
-          <frame_name>${name}_link</frame_name>
+          <frame_name>${name}_ray_link</frame_name>
         </plugin>
       </sensor>
     </gazebo>
-        <joint name="${name}_hokuyo_urg_lidar_mount_joint" type="fixed">
-            <xacro:insert_block name="origin"/>
-            <parent link="${parent}"/>
-            <child link="${name}_hokuyo_urg_lidar_link"/>
-        </joint>
-    </xacro:macro>
+  </xacro:macro>
 </robot>

File: urdf/skratch_urdf.xacro (robot description, xacro)
@@ -38,9 +38,9 @@
         <origin xyz="-0.190 -0.118 0.0" rpy="0.0 0.0 0.0"/>
     </xacro:kelo_drive_top>
-    <!-- LIDAR Mounting -->
-    <xacro:lidar_mount name="front" parent="skratch_base" ros_topic="/scan_front" update_rate="10" min_angle="0.0" max_angle="-3.14">
+    <!-- Lidar Mount -->
+    <xacro:lidar_mount name="front" parent="skratch_base">
         <origin xyz="0.272 -0.158 0.1416" rpy="0.0 0.0 0.0"/>
     </xacro:lidar_mount>
-    <xacro:lidar_mount name="rear" parent="skratch_base" ros_topic="/scan_rear" update_rate="10" min_angle="0.0" max_angle="-3.14">
+    <xacro:lidar_mount name="rear" parent="skratch_base">
         <origin xyz="-0.272 0.167 0.1416" rpy="0.0 0.0 3.14"/>
     </xacro:lidar_mount>
