Commit message: Updating the package in a foormat

File: description/sensor_mounts/lidar_mount.xacro (robot description, xacro)
@@ -9,5 +9,5 @@
 <robot name="lidar_mount" xmlns:xacro="http://www.ros.org/wiki/xacro">
     <xacro:macro name="lidar_mount" params="name parent *origin">
-        <xacro:include filename="$(find skratch_description)/sensors/hokuyo_urg_04lx_ug01.xacro"/>
+        <xacro:include filename="$(find skratch_description)/description/sensors/hokuyo_urg_04lx_ug01.xacro"/>
         <link name="${name}_lidar_mount">
             <inertial>

File: description/wheels/kelo_drive_mid.urdf.xacro (robot description, xacro)
@@ -5,4 +5,6 @@
 Author:
 Sushant Chavan
+Maintainer:
+Chaitanya Gumudala
 This software is published under a dual-license: GNU Lesser General Public
 License LGPL 2.1 and BSD license. The dual-license implies that users of this
@@ -30,19 +32,42 @@
 -->
 <robot xmlns:xacro="http://www.ros.org/wiki/xacro">
-    <xacro:macro name="kelo_drive_wheel" params="name parent *origin movable_joints:=true">
-        <xacro:include filename="$(find skratch_description)/wheels/common.xacro" />
+    <xacro:macro name="kelo_drive_mid" params="name parent *origin movable_joints:=true">
+        <xacro:include filename="$(find skratch_description)/description/wheels/common.xacro" />
+        <xacro:include filename="$(find skratch_description)/description/wheels/kelo_drive_wheel.urdf.xacro" />
+        <!-- PIVOT Link-->
+        <link name="${name}_pivot_link">
+            <visual>
+                <origin xyz="0 0 0" rpy="0 0 0"/>
+                <geometry>
+                    <mesh filename="file://$(find skratch_description)/meshes/kelo_drive/kelo_drive_mid_part.dae" scale="1 1 1"/>
+                </geometry>
+            </visual>
+            <collision>
+                <origin xyz="0 0 0" rpy="0 0 0"/>
+                <geometry>
+                    <mesh filename="file://$(find skratch_description)/meshes/kelo_drive/kelo_drive_mid_part.dae" scale="1 1 1"/>
+                </geometry>
+            </collision>
+            <inertial>
+                <origin xyz="0.00023 -0.00095 0.04843" rpy="0 0 0"/>
+                <mass value="1.46273"/>
+                <inertia ixx="0.00302046423" ixy="0.00000851844" ixz="0.00001188180" iyy="0.00326495472" iyz="0.00001855408" izz="0.00386072964"/>
+            </inertial>
+        </link>
+        <!-- PIVOT continous or fixed-->
         <xacro:if value="${movable_joints}">
-            <joint name="${name}_joint" type="continuous">
+            <joint name="${name}_pivot_joint" type="continuous">
                 <xacro:insert_block name="origin" />
-                <axis xyz="0 1 0"/>
+                <axis xyz="0 0 1"/>
                 <parent link="${parent}"/>
-                <child link="${name}_link" />
+                <child link="${name}_pivot_link" />
+                <limit effort="2.0" velocity="1.0"/>
             </joint>
-            <transmission name="${name}_transmission">
+            <transmission name="${name}_pivot_transmission">
                 <type>transmission_interface/SimpleTransmission</type>
-                <joint name="${name}_joint">
+                <joint name="${name}_pivot_joint">
                     <hardwareInterface>hardware_interface/EffortJointInterface</hardwareInterface>
                 </joint>
-                <actuator name="${name}_motor">
+                <actuator name="${name}_pivot_motor">
                     <hardwareInterface>hardware_interface/EffortJointInterface</hardwareInterface>
                     <mechanicalReduction>1</mechanicalReduction>
@@ -51,30 +76,19 @@
         </xacro:if>
         <xacro:unless value="${movable_joints}">
-            <joint name="${name}_joint" type="fixed">
+            <joint name="${name}_pivot_joint" type="fixed">
                 <xacro:insert_block name="origin" />
-                <axis xyz="0 1 0"/>
+                <axis xyz="0 0 1"/>
                 <parent link="${parent}"/>
-                <child link="${name}_link" />
+                <child link="${name}_pivot_link" />
             </joint>
         </xacro:unless>
-        <link name="${name}_link">
-            <visual>
-                <origin xyz="0 0 0" rpy="0 0 0"/>
-                <geometry>
-                    <mesh filename="file://$(find skratch_description)/meshes/kelo_drive/kelo_drive_wheel.stl" scale="1 1 1"/>
-                </geometry>
-            </visual>
-            <collision>
-                <origin xyz="0 0 0" rpy="0 0 0"/>
-                <geometry>
-                    <mesh filename="file://$(find skratch_description)/meshes/kelo_drive/kelo_drive_wheel.stl" scale="1 1 1"/>
-                </geometry>
-            </collision>
-             <inertial>
-                <origin xyz="0 0 0" rpy="0 0 0"/>
-                <mass value="1.56317"/>
-                <inertia ixx="0.00101253363" ixy="0.00000000000" ixz="0.00000001020" iyy="0.00157998524" iyz="-0.00000055474" izz="0.00101282739"/>
-            </inertial>
-        </link>
+        <!-- LEFT HUB WHEEL -->
+        <xacro:kelo_drive_wheel name="${name}_left_hub_wheel" parent="${name}_pivot_link" movable_joints="${movable_joints}">
+            <origin xyz="-0.01 0.039326 0.001514" rpy="0 0 0.0"/>
+        </xacro:kelo_drive_wheel>
+        <!-- RIGHT HUB WHEEL -->
+        <xacro:kelo_drive_wheel name="${name}_right_hub_wheel" parent="${name}_pivot_link" movable_joints="${movable_joints}">
+            <origin xyz="-0.01 -0.039326 0.001514" rpy="0 0 0.0"/>
+        </xacro:kelo_drive_wheel>
     </xacro:macro>
 </robot>

File: description/wheels/kelo_drive_top.urdf.xacro (robot description, xacro)
@@ -8,5 +8,5 @@
 <robot xmlns:xacro="http://www.ros.org/wiki/xacro">
   <!-- Include the mid part macro -->
-  <xacro:include filename="$(find skratch_description)/wheels/kelo_drive_mid.urdf.xacro" />
+  <xacro:include filename="$(find skratch_description)/description/wheels/kelo_drive_mid.urdf.xacro" />
   <!--
     Macro for full KELO drive:

File: description/wheels/kelo_drive_wheel.urdf.xacro (robot description, xacro)
@@ -5,6 +5,4 @@
 Author:
 Sushant Chavan
-Maintainer:
-Chaitanya Gumudala
 This software is published under a dual-license: GNU Lesser General Public
 License LGPL 2.1 and BSD license. The dual-license implies that users of this
@@ -32,42 +30,19 @@
 -->
 <robot xmlns:xacro="http://www.ros.org/wiki/xacro">
-    <xacro:macro name="kelo_drive_mid" params="name parent *origin movable_joints:=true">
-        <xacro:include filename="$(find skratch_description)/wheels/common.xacro" />
-        <xacro:include filename="$(find skratch_description)/wheels/kelo_drive_wheel.urdf.xacro" />
-        <!-- PIVOT Link-->
-        <link name="${name}_pivot_link">
-            <visual>
-                <origin xyz="0 0 0" rpy="0 0 0"/>
-                <geometry>
-                    <mesh filename="file://$(find skratch_description)/meshes/kelo_drive/kelo_drive_mid_part.dae" scale="1 1 1"/>
-                </geometry>
-            </visual>
-            <collision>
-                <origin xyz="0 0 0" rpy="0 0 0"/>
-                <geometry>
-                    <mesh filename="file://$(find skratch_description)/meshes/kelo_drive/kelo_drive_mid_part.dae" scale="1 1 1"/>
-                </geometry>
-            </collision>
-            <inertial>
-                <origin xyz="0.00023 -0.00095 0.04843" rpy="0 0 0"/>
-                <mass value="1.46273"/>
-                <inertia ixx="0.00302046423" ixy="0.00000851844" ixz="0.00001188180" iyy="0.00326495472" iyz="0.00001855408" izz="0.00386072964"/>
-            </inertial>
-        </link>
-        <!-- PIVOT continous or fixed-->
+    <xacro:macro name="kelo_drive_wheel" params="name parent *origin movable_joints:=true">
+        <xacro:include filename="$(find skratch_description)/description/wheels/common.xacro" />
         <xacro:if value="${movable_joints}">
-            <joint name="${name}_pivot_joint" type="continuous">
+            <joint name="${name}_joint" type="continuous">
                 <xacro:insert_block name="origin" />
-                <axis xyz="0 0 1"/>
+                <axis xyz="0 1 0"/>
                 <parent link="${parent}"/>
-                <child link="${name}_pivot_link" />
-                <limit effort="2.0" velocity="1.0"/>
+                <child link="${name}_link" />
             </joint>
-            <transmission name="${name}_pivot_transmission">
+            <transmission name="${name}_transmission">
                 <type>transmission_interface/SimpleTransmission</type>
-                <joint name="${name}_pivot_joint">
+                <joint name="${name}_joint">
                     <hardwareInterface>hardware_interface/EffortJointInterface</hardwareInterface>
                 </joint>
-                <actuator name="${name}_pivot_motor">
+                <actuator name="${name}_motor">
                     <hardwareInterface>hardware_interface/EffortJointInterface</hardwareInterface>
                     <mechanicalReduction>1</mechanicalReduction>
@@ -76,19 +51,30 @@
         </xacro:if>
         <xacro:unless value="${movable_joints}">
-            <joint name="${name}_pivot_joint" type="fixed">
+            <joint name="${name}_joint" type="fixed">
                 <xacro:insert_block name="origin" />
-                <axis xyz="0 0 1"/>
+                <axis xyz="0 1 0"/>
                 <parent link="${parent}"/>
-                <child link="${name}_pivot_link" />
+                <child link="${name}_link" />
             </joint>
         </xacro:unless>
-        <!-- LEFT HUB WHEEL -->
-        <xacro:kelo_drive_wheel name="${name}_left_hub_wheel" parent="${name}_pivot_link" movable_joints="${movable_joints}">
-            <origin xyz="-0.01 0.039326 0.001514" rpy="0 0 0.0"/>
-        </xacro:kelo_drive_wheel>
-        <!-- RIGHT HUB WHEEL -->
-        <xacro:kelo_drive_wheel name="${name}_right_hub_wheel" parent="${name}_pivot_link" movable_joints="${movable_joints}">
-            <origin xyz="-0.01 -0.039326 0.001514" rpy="0 0 0.0"/>
-        </xacro:kelo_drive_wheel>
+        <link name="${name}_link">
+            <visual>
+                <origin xyz="0 0 0" rpy="0 0 0"/>
+                <geometry>
+                    <mesh filename="file://$(find skratch_description)/meshes/kelo_drive/kelo_drive_wheel.stl" scale="1 1 1"/>
+                </geometry>
+            </visual>
+            <collision>
+                <origin xyz="0 0 0" rpy="0 0 0"/>
+                <geometry>
+                    <mesh filename="file://$(find skratch_description)/meshes/kelo_drive/kelo_drive_wheel.stl" scale="1 1 1"/>
+                </geometry>
+            </collision>
+             <inertial>
+                <origin xyz="0 0 0" rpy="0 0 0"/>
+                <mass value="1.56317"/>
+                <inertia ixx="0.00101253363" ixy="0.00000000000" ixz="0.00000001020" iyy="0.00157998524" iyz="-0.00000055474" izz="0.00101282739"/>
+            </inertial>
+        </link>
     </xacro:macro>
 </robot>

File: urdf/skratch_urdf.xacro (robot description, xacro)
@@ -5,8 +5,8 @@
     <xacro:arg name="use_sim" default="true"/>
     <!--Include necessary xacros-->
-    <xacro:include filename="$(find skratch_description)/base/skratch_base.xacro" />
-    <xacro:include filename="$(find skratch_description)/wheels/kelo_drive_top.urdf.xacro" />
-    <xacro:include filename="$(find skratch_description)/sensor_mounts/lidar_mount.xacro"/>
-    <xacro:include filename="$(find skratch_description)/base/kinova_arm_base_plate.xacro"/>
+    <xacro:include filename="$(find skratch_description)/description/base/skratch_base.xacro" />
+    <xacro:include filename="$(find skratch_description)/description/wheels/kelo_drive_top.urdf.xacro" />
+    <xacro:include filename="$(find skratch_description)/description/sensor_mounts/lidar_mount.xacro"/>
+    <xacro:include filename="$(find skratch_description)/description/base/kinova_arm_base_plate.xacro"/>
     <!-- Start building the robot -->
     <link name="base_link"/>
