Commit message: [URDF] reducing lidar height, to get 5 cm workspace

File: description/sensors/hokuyo_urg_04lx_ug01.xacro (robot description, xacro)
@@ -39,5 +39,5 @@
     <!-- ↓↓↓ Move ray start point 5 cm below STL origin ↓↓↓ -->
     <joint name="${name}_ray_joint" type="fixed">
-      <origin xyz="0 0 -0.05" rpy="0 0 0"/>
+      <origin xyz="0 0 -0.06" rpy="0 0 0"/>
       <parent link="${name}_stl_link"/>
       <child link="${name}_ray_link"/>
